Commit message: Added sonar to uwrosys-launch file.

File: uuv_descriptions/robots/rexrov_oberon4.xacro (robot description, xacro)
@@ -15,4 +15,5 @@
   <xacro:arg name="debug" default="0"/>
   <xacro:arg name="namespace" default="rexrov"/>
+  <xacro:arg name="config" default="base"/>
   <xacro:arg name="inertial_reference_frame" default="world"/>
   <!-- Include the ROV macro file -->
@@ -40,4 +41,10 @@
     <origin xyz="1.3 0.5 -0.615" rpy="0 0 0"/>
   </xacro:oberon4>
+  <xacro:property name="sensor_config" value="$(arg config)"/>
+  <xacro:if value="${sensor_config == 'sonar'}">
+    <xacro:forward_multibeam_sonar_m450_130 namespace="$(arg namespace)" parent_link="$(arg namespace)/base_link">
+      <origin xyz="1.4 0 0.65" rpy="0 0 0"/>
+    </xacro:forward_multibeam_sonar_m450_130>
+ </xacro:if>
   <gazebo>
       <plugin name="gazebo_ros_control" filename="libgazebo_ros_control.so">

Commit message: Removed multibeam config from Oberon4 config.

File: uuv_descriptions/robots/rexrov_oberon4.xacro (robot description, xacro)
@@ -41,10 +41,4 @@
     <origin xyz="1.3 0.5 -0.615" rpy="0 0 0"/>
   </xacro:oberon4>
-  <xacro:property name="sensor_config" value="$(arg config)"/>
-  <xacro:if value="${sensor_config == 'sonar'}">
-    <xacro:forward_multibeam_sonar_m450_130 namespace="$(arg namespace)" parent_link="$(arg namespace)/base_link">
-      <origin xyz="1.4 0 0.65" rpy="0 0 0"/>
-    </xacro:forward_multibeam_sonar_m450_130>
- </xacro:if>
   <gazebo>
       <plugin name="gazebo_ros_control" filename="libgazebo_ros_control.so">

Commit message: Fixed sonar output.

File: uuv_descriptions/robots/rexrov_oberon4.xacro (robot description, xacro)
@@ -41,4 +41,10 @@
     <origin xyz="1.3 0.5 -0.615" rpy="0 0 0"/>
   </xacro:oberon4>
+  <!--<xacro:property name="sensor_config" value="$(arg config)"/>
+    <xacro:if value="${sensor_config == 'sonar'}">-->
+  <xacro:forward_multibeam_sonar_m450_130 namespace="$(arg namespace)" parent_link="$(arg namespace)/base_link">
+    <origin xyz="1.4 0 0.65" rpy="0 0 0"/>
+  </xacro:forward_multibeam_sonar_m450_130>
+  <!--</xacro:if>-->
   <gazebo>
       <plugin name="gazebo_ros_control" filename="libgazebo_ros_control.so">
